File: mainboard/mainboard/mainboard.kicad_pcb (KiCad board)
At the start: 2 copper layers, 17 parts, among them J1_btcomms_1 Conn_01x06, J2_IMU1 Conn_01x08, J3_hoverboard_serial1 Conn_01x03, J5_LEFT_HALL_IN1 Conn_01x04, J6_RIGHT_HALL_IN1 Conn_01x04, J7_btcomms_2 Conn_01x06, U1 STM32F446RETx

Commit message: ready for first cut
Parts:
- added H1: MountingHole, MountingHole:MountingHole_3.2mm_M3, B.Cu at (55.3, 67.8)
- added H2: MountingHole, MountingHole:MountingHole_3.2mm_M3, B.Cu at (55.3, 153.4)
- added H3: MountingHole, MountingHole:MountingHole_3.2mm_M3, B.Cu at (132.0, 153.4)
- added J4_serial3: Conn_01x04, kicad_footprints:Molex_KK-254_AE-6410-04A_1x04_P2.54mm_Vertical, B.Cu at (56.6, 78.0)
- C1, C2, C3, C4, C5, C6, U1: moved to B.Cu
- J1_btcomms_1, J7_btcomms_2: footprint Connector_Molex:Molex_KK-254_AE-6410-06A_1x06_P2.54mm_Vertical -> kicad_footprints:Molex_KK-254_AE-6410-06A_1x06_P2.54mm_Vertical; moved to B.Cu
- J2_IMU1: footprint Connector_Molex:Molex_KK-254_AE-6410-08A_1x08_P2.54mm_Vertical -> kicad_footprints:Molex_KK-254_AE-6410-08A_1x08_P2.54mm_Vertical; moved to B.Cu
- J3_hoverboard_serial1: footprint Connector_Molex:Molex_KK-254_AE-6410-03A_1x03_P2.54mm_Vertical -> kicad_footprints:Molex_KK-254_AE-6410-03A_1x03_P2.54mm_Vertical; moved to B.Cu
- J5_LEFT_HALL_IN1, J6_RIGHT_HALL_IN1: footprint Connector_Molex:Molex_KK-254_AE-6410-04A_1x04_P2.54mm_Vertical -> kicad_footprints:Molex_KK-254_AE-6410-04A_1x04_P2.54mm_Vertical; moved to B.Cu
- R1, R2, R3, R4: footprint Resistor_THT:R_Axial_DIN0204_L3.6mm_D1.6mm_P5.08mm_Horizontal -> kicad_footprints:R_Axial_DIN0204_L3.6mm_D1.6mm_P5.08mm_Horizontal; moved to B.Cu
- moved J2_IMU1 99.9 mm to (56.6, 97.0)
- moved J7_btcomms_2 99.9 mm to (56.6, 130.8)
- moved R4 89.8 mm to (61.7, 142.2)
- moved R3 71.1 mm to (71.1, 142.2)
- moved C3 58.6 mm to (77.4, 139.5), turned to 0 degrees
- moved C5 58.6 mm to (77.4, 142.8), turned to 0 degrees
- moved C1 58.4 mm to (77.5, 136.2), turned to 0 degrees
- moved J5_LEFT_HALL_IN1 49.1 mm to (82.2, 153.3), turned to 180 degrees
- moved U1 46.0 mm to (128.7, 99.1), turned to 180 degrees
- moved C6 41.2 mm to (86.3, 135.4), turned to 0 degrees
- moved C4 36.3 mm to (88.8, 132.1), turned to 0 degrees
- moved C2 31.5 mm to (91.4, 129.0), turned to 0 degrees
- moved J6_RIGHT_HALL_IN1 26.7 mm to (93.9, 153.3), turned to 180 degrees
- moved J3_hoverboard_serial1 22.4 mm to (116.3, 153.2), turned to 0 degrees
- moved R1 16.0 mm to (112.5, 118.9)
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Connections:
- J1_btcomms_1 pad 1: (no net) -> Net-(J1_btcomms_1-Pad1)
- J1_btcomms_1 pad 6: (no net) -> Net-(J1_btcomms_1-Pad6)
- J2_IMU1 pad 5: (no net) -> Net-(J2_IMU1-Pad5)
- J2_IMU1 pad 6: (no net) -> Net-(J2_IMU1-Pad6)
- J2_IMU1 pad 7: (no net) -> Net-(J2_IMU1-Pad7)
- J7_btcomms_2 pad 1: (no net) -> Net-(J7_btcomms_2-Pad1)
- J7_btcomms_2 pad 6: (no net) -> Net-(J7_btcomms_2-Pad6)
- U1 pad BOOT0: (no net) -> Net-(U1-PadBOOT0)
- U1 pad PA11: (no net) -> Net-(U1-PadPA11)
- U1 pad PA12: (no net) -> Net-(U1-PadPA12)
- U1 pad PA13: (no net) -> Net-(U1-PadPA13)
- U1 pad PA14: (no net) -> Net-(U1-PadPA14)
- U1 pad PA15: (no net) -> Net-(U1-PadPA15)
- U1 pad PA4: (no net) -> Net-(U1-PadPA4)
- U1 pad PA5: (no net) -> Net-(U1-PadPA5)
- U1 pad PA6: (no net) -> Net-(U1-PadPA6)
- U1 pad PA7: (no net) -> Net-(U1-PadPA7)
- U1 pad PB0: (no net) -> Net-(U1-PadPB0)
- U1 pad PB1: (no net) -> Net-(U1-PadPB1)
- U1 pad PB10: (no net) -> Net-(U1-PadPB10)
- U1 pad PB12: (no net) -> Net-(U1-PadPB12)
- U1 pad PB13: (no net) -> Net-(U1-PadPB13)
- U1 pad PB14: (no net) -> Net-(U1-PadPB14)
- U1 pad PB15: (no net) -> Net-(U1-PadPB15)
- U1 pad PB2: (no net) -> Net-(U1-PadPB2)
- U1 pad PB6: (no net) -> Net-(U1-PadPB6)
- U1 pad PB7: (no net) -> Net-(U1-PadPB7)
- U1 pad PC0: (no net) -> Net-(U1-PadPC0)
- U1 pad PC1: (no net) -> Net-(U1-PadPC1)
- U1 pad PC10: (no net) -> serial3_Rx
- U1 pad PC11: (no net) -> serial3_Tx
- U1 pad PC13: (no net) -> Net-(U1-PadPC13)
- U1 pad PC14: (no net) -> Net-(U1-PadPC14)
- U1 pad PC15: (no net) -> Net-(U1-PadPC15)
- U1 pad PC2: (no net) -> Net-(U1-PadPC2)
- U1 pad PC3: (no net) -> Net-(U1-PadPC3)
- U1 pad PC4: (no net) -> Net-(U1-PadPC4)
- U1 pad PC5: (no net) -> Net-(U1-PadPC5)
- U1 pad PC6: (no net) -> Net-(U1-PadPC6)
- U1 pad PC8: (no net) -> Net-(U1-PadPC8)
- U1 pad PC9: (no net) -> Net-(U1-PadPC9)
- U1 pad PH0: (no net) -> Net-(U1-PadPH0)
- U1 pad PH1: (no net) -> Net-(U1-PadPH1)
- U1 pad VBAT: (no net) -> Net-(U1-PadVBAT)
- U1 pad VDD: (no net) -> Net-(U1-PadVDD)
Routing:
- net GND: track 378.6 -> 535.4 mm
- net serial3_Rx: track 0.00 -> 82.4 mm
- net serial3_Tx: track 0.00 -> 76.2 mm
- net R_hall_A_LPF: track 19.9 -> 38.6 mm
- net bluetooth_serial_1_Rx: track 45.5 -> 59.1 mm, vias 0 -> 2
- net +5V: track 230.0 -> 233.6 mm
Other:
- board outline added: 90.2 x 99.1 mm
- net class Default: via_dia 1.2 -> 1.7
- net class top_thin removed
- rule trace_min: 0.2 -> 0.6
- rule via_min_size: 0.4 -> 0.8
